Commit message: fix
Integrate namespace

File: urdf/dream_walker.urdf (robot description, URDF)
Before this commit: robot dw_descliption3, 18 links, 17 joints
Links:
- link A0_Link: geometry collision mesh filename=package://dream_walker/meshes/A0_Link.STL; visual mesh filename=package://dream_walker/meshes/A0_Link.STL
- link A1_Link: geometry collision mesh filename=package://dream_walker/meshes/A1_Link.STL; visual mesh filename=package://dream_walker/meshes/A1_Link.STL
- link A2_Link: geometry collision mesh filename=package://dream_walker/meshes/A2_Link.STL; visual mesh filename=package://dream_walker/meshes/A2_Link.STL
- link A3_Link: geometry collision mesh filename=package://dream_walker/meshes/A3_Link.STL; visual mesh filename=package://dream_walker/meshes/A3_Link.STL
- link B0_Link: geometry collision mesh filename=package://dream_walker/meshes/B0_Link.STL; visual mesh filename=package://dream_walker/meshes/B0_Link.STL
- link B1_Link: geometry collision mesh filename=package://dream_walker/meshes/B1_Link.STL; visual mesh filename=package://dream_walker/meshes/B1_Link.STL
- link B2_Link: geometry collision mesh filename=package://dream_walker/meshes/B2_Link.STL; visual mesh filename=package://dream_walker/meshes/B2_Link.STL
- link B3_Link: geometry collision mesh filename=package://dream_walker/meshes/B3_Link.STL; visual mesh filename=package://dream_walker/meshes/B3_Link.STL
- link C0_Link: geometry collision mesh filename=package://dream_walker/meshes/C0_Link.STL; visual mesh filename=package://dream_walker/meshes/C0_Link.STL
- link C1_Link: geometry collision mesh filename=package://dream_walker/meshes/C1_Link.STL; visual mesh filename=package://dream_walker/meshes/C1_Link.STL
- link C2_Link: geometry collision mesh filename=package://dream_walker/meshes/C2_Link.STL; visual mesh filename=package://dream_walker/meshes/C2_Link.STL
- link C3_Link: geometry collision mesh filename=package://dream_walker/meshes/C3_Link.STL; visual mesh filename=package://dream_walker/meshes/C3_Link.STL
- link D0_Link: geometry collision mesh filename=package://dream_walker/meshes/D0_Link.STL; visual mesh filename=package://dream_walker/meshes/D0_Link.STL
- link D1_Link: geometry collision mesh filename=package://dream_walker/meshes/D1_Link.STL; visual mesh filename=package://dream_walker/meshes/D1_Link.STL
- link D2_Link: geometry collision mesh filename=package://dream_walker/meshes/D2_Link.STL; visual mesh filename=package://dream_walker/meshes/D2_Link.STL
- link D3_Link: geometry collision mesh filename=package://dream_walker/meshes/D3_Link.STL; visual mesh filename=package://dream_walker/meshes/D3_Link.STL
- link base_link: geometry collision mesh filename=package://dream_walker/meshes/base_link.STL; visual mesh filename=package://dream_walker/meshes/base_link.STL

Commit message: update
changed the axis parameter to boolean type

File: urdf/dream_walker.urdf (robot description, URDF)
Before this commit: robot dream_walker, 18 links, 17 joints
Joints:
- joint A1_joint: axis 0.078459 0.99692 0 -> 0 1 0
- joint B1_joint: axis 0.078459 0.99692 0 -> 0 1 0
- joint C1_joint: axis 0.078459 0.99692 0 -> 0 1 0
- joint D1_joint: axis 0.078459 0.99692 0 -> 0 1 0

Commit message: update
changed joint origin parameter

File: urdf/dream_walker.urdf (robot description, URDF)
Before this commit: robot dream_walker, 18 links, 17 joints
Joints:
- joint A0_joint: origin xyz=0.3 -0.083 0.55565 rpy=-1.5708 0 -1.5708 -> xyz=0.3 -0.083 0.55565 rpy=-1.57079632679 0 -1.57079632679
- joint A1_joint: origin xyz=0 0 0 rpy=-1.5708 0.07854 -1.5708 -> xyz=0 0 0 rpy=-1.57079632679 0.07854 -1.57079632679
- joint A3_joint: origin xyz=0 -0.32 0.135 rpy=0 0 1.5708 -> xyz=0 -0.32 0.135 rpy=0 0 1.57079632679
- joint B0_joint: origin xyz=0.3 0.083 0.55565 rpy=-1.5708 0 -1.5708 -> xyz=0.3 0.083 0.55565 rpy=-1.57079632679 0 -1.57079632679
- joint B1_joint: origin xyz=0 0 0 rpy=-1.5708 0.07854 1.5708 -> xyz=0 0 0 rpy=-1.57079632679 0.07854 1.57079632679
- joint B3_joint: origin xyz=0 -0.32 0.135 rpy=0 0 -1.5708 -> xyz=0 -0.32 0.135 rpy=0 0 -1.57079632679
- joint C0_joint: origin xyz=-0.3 -0.083 0.55565 rpy=1.5708 0 -1.5708 -> xyz=-0.3 -0.083 0.55565 rpy=1.57079632679 0 -1.57079632679
- joint C1_joint: origin xyz=0 0 0 rpy=-1.5708 0.07854 -1.5708 -> xyz=0 0 0 rpy=-1.57079632679 0.07854 -1.57079632679
- joint C3_joint: origin xyz=0 -0.32 0.135 rpy=0 0 1.5708 -> xyz=0 -0.32 0.135 rpy=0 0 1.57079632679
- joint D0_joint: origin xyz=-0.3 0.083 0.55565 rpy=1.5708 0 -1.5708 -> xyz=-0.3 0.083 0.55565 rpy=1.57079632679 0 -1.57079632679
- joint D1_joint: origin xyz=0 0 0 rpy=-1.5708 0.07854 1.5708 -> xyz=0 0 0 rpy=-1.57079632679 0.07854 1.57079632679
- joint D3_joint: origin xyz=0 -0.32 0.135 rpy=0 0 -1.5708 -> xyz=0 -0.32 0.135 rpy=0 0 -1.57079632679

Commit message: update
changed rotation limit.and dynamics raram are all zero.

File: urdf/dream_walker.urdf (robot description, URDF)
Before this commit: robot dream_walker, 18 links, 17 joints
Joints:
- joint A1_joint: limit lower=-1.5075 upper=1.5075 effort=1000 velocity=1000 -> lower=-9.42 upper=9.42 effort=1000 velocity=1000
- joint A2_joint: limit lower=-1.5075 upper=1.5075 effort=1000 velocity=1000 -> lower=-9.42 upper=9.42 effort=1000 velocity=1000
- joint A3_joint: limit lower=-1.5075 upper=1.5075 effort=1000 velocity=1000 -> lower=-9.42 upper=9.42 effort=1000 velocity=1000
- joint B1_joint: limit lower=-1.5075 upper=1.5075 effort=1000 velocity=1000 -> lower=-9.42 upper=9.42 effort=1000 velocity=1000
- joint B2_joint: limit lower=-1.5075 upper=1.5075 effort=1000 velocity=1000 -> lower=-9.42 upper=9.42 effort=1000 velocity=1000
- joint B3_joint: limit lower=-1.5075 upper=1.5075 effort=1000 velocity=1000 -> lower=-9.42 upper=9.42 effort=1000 velocity=1000
- joint C1_joint: limit lower=-1.5075 upper=1.5075 effort=1000 velocity=1000 -> lower=-9.42 upper=9.42 effort=1000 velocity=1000
- joint C2_joint: limit lower=-1.5075 upper=1.5075 effort=1000 velocity=1000 -> lower=-9.42 upper=9.42 effort=1000 velocity=1000
- joint C3_joint: limit lower=-1.5075 upper=1.5075 effort=1000 velocity=1000 -> lower=-9.42 upper=9.42 effort=1000 velocity=1000
- joint D1_joint: limit lower=-1.5075 upper=1.5075 effort=1000 velocity=1000 -> lower=-9.42 upper=9.42 effort=1000 velocity=1000
- joint D2_joint: limit lower=-1.5075 upper=1.5075 effort=1000 velocity=1000 -> lower=-9.42 upper=9.42 effort=1000 velocity=1000
- joint D3_joint: limit lower=-1.5075 upper=1.5075 effort=1000 velocity=1000 -> lower=-9.42 upper=9.42 effort=1000 velocity=1000
